Commit message: Feat: add scripts for using vr control koch arm

File: Assets/model/koch_arm/koch_arm_unity.urdf (robot description, URDF)
Before this commit: robot koch_arm, 7 links, 6 joints
Joints:
- joint joint4: origin xyz=0.000125 0.090467 0.002747 rpy=0 0 0 -> xyz=0.000125 0.090467 0.002747 rpy=1.57 0 0
